File: Pcb/Blue_way_V1.0/MCU.kicad_sch (KiCad schematic)
At the start: 0 parts

Commit message: BNO085 Schematic updated
Other:
- company: (none) -> BlueWay Horizon
- title: (none) -> Avionics Subsystem
Changed lines of the file:
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@@
 	(generator_version "9.0")
 	(paper "A4")
+	(title_block
+		(title "Avionics Subsystem")
+		(date "2026-03-05")
+		(rev "0.0.1")
+		(company "BlueWay Horizon")
+		(comment 1 "www.bluewayhorizon.in")
+	)
 )
