File: Pcb/Blue_way_V1.0/BNO085.kicad_sch (KiCad schematic)
At the start: 23 parts, among them IC1 74HC4050DB,118, Q1 BSS138, Q2 BSS138, U1 BNO085, Y1 32.768kHz

Commit message: SHT and BMP Added with LoRa Comm Module
Parts:
- renumbered D1 to BNO_085
Changed lines of the file:
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@@
 		(dnp no)
 		(fields_autoplaced yes)
-		(property "Reference" "D1"
+		(property "Reference" "BNO_085"
 			(at 149.86 130.7464 90)
 			(effects
@@
 			(project ""
 				(path "/2f3247fa-a7e8-4139-878f-1aed25c1e4d8/7dab7a21-a5d5-4af2-99e9-1daf90182840/181386e5-10e9-4c7a-bc71-286646d180c9"
-					(reference "D1")
+					(reference "BNO_085")
 					(unit 1)
 				)
